File: Hardware/KiCad Source Files/Power.kicad_sch (KiCad schematic)
At the start: 15 parts, among them U1 MC33063AP

Commit message: V3 connector board: strobe pulse limiter, USB-C fixes, boost protection
Mechanical: board outline, all mounting/tab/breakaway holes and every
existing part position are unchanged (checked against the previous revision);
all new parts are on the top side and no taller than existing parts.
PiTrac software compatibility: the LED current-control circuit and the
DAC/ADC/DIAG interface used by strobe_calibration_manager.py are unchanged.

Strobe (CC Sink sheet)
- AC-coupled pulse limiter: TRIG (DIAG/MOSI via D3/D4) -> C16 220nF ->
  GATE-DRV, R28 10K to GND (tau 2.2 ms). 8.7-130 us strobes and the
  calibration pulse pass (guaranteed >= ~0.38 ms by the MCP1407 input
  limits); a stuck-high DIAG turns the driver off after ~1.7 ms typical,
  <= ~2.8 ms worst case, so 10 A can no longer be held on.

USB-C (Connectors sheet, USB4085-GF-A footprint)
- J2/J5 feed 5 V to the Pis: add 10K Rp on CC1/CC2 (R24-R27, 1206).
- Footprint rebuilt to GCT's land pattern (16 plated 0.40/0.66 mm pins).
  The old VBUS/GND pads had 0.1 mm top-side copper (annular-ring DRC
  errors; Pi supply current only reached them via the barrel/bottom pad).

Boost (Power sheet)
- F1 MF-MSMF050-2 polyfuse in the boost input only (+5V_BST: C1/C2/C3/R1/
  U1); PCB: +5V_BST F.Cu island, +5V B.Cu bridge keeps the Pi feed width.
- D16 P4SMA39CA clamp on VIR (open-feedback fault; relies on F1).
- R5 2K49 -> 10K (was ~0.45 W in a 1/4 W resistor).

Housekeeping
- Project sym/fp-lib-tables; USB4085-GF-A added to the symbol library;
  pin types for custom parts; locally modified Q_NPN/Q_NMOS/LED moved into
  the project library (Q_NPN_EBC, Q_NMOS_SGD, LED_ThermalPad) to keep their
  numeric pinouts; no-connect flags; PWR_FLAGs; GATE-DRV wire to Q3 fixed.
- ERC pin map (project-wide): open emitter on a power rail allowed
  (MC33063 SwE to GND).
- Add V3 Connector Only.kicad_pro (board had no rules; DRC used defaults).
- Breakaway holes marked board-only.
- Regenerated Gerber/drill zips, BOM and centroid CSVs (same for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
Parts:
- added D16: P4SMA39CA, Diode_SMD:D_SMA, symbol Device:D_TVS
- added F1: 0.5A hold, Fuse:Fuse_1812_4532Metric_Pad1.30x3.40mm_HandSolder, symbol Device:Polyfuse
- R5: value 2K49 -> 10K; Part Number MFR-25FTE52-2K49 -> MFR-25FRF52-10K
Connections:
- net +5V: now also F1.1; no longer C1.1, C2.1, C3.1, R1.2, U1.6 (Vin)
- net GND: now also D16.2 (A2)
- net VIR: now also D16.1 (A1)
- new net +5V_BST: C1.1, C2.1, C3.1, F1.2, R1.2, U1.6 (Vin)
Other:
- note added: "Protection (added). F1: resettable fuse in the boost input only (not in the +5V path to the Pis). It limits a VIR short (e.g. C6, D16 or an LED/MOSFET failing short), which the MC33063 current limit cannot stop because current flows 5V > R1 > L1 > D1 directly. D16: clamps VIR if the feedback divider (R3/R4) opens. VBR(min) 37.1 V is above worst-case normal VIR (~36.8 V). It is a clamp-then-fail-s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"
