File: Hardware/KiCad Source Files/DAC.kicad_sch (KiCad schematic)
At the start: 14 parts, among them U4 LM4040LP-2.0, U5 MCP4801

Commit message: V3 connector board: strobe pulse limiter, USB-C fixes, boost protection
Mechanical: board outline, all mounting/tab/breakaway holes and every
existing part position are unchanged (checked against the previous revision);
all new parts are on the top side and no taller than existing parts.
PiTrac software compatibility: the LED current-control circuit and the
DAC/ADC/DIAG interface used by strobe_calibration_manager.py are unchanged.

Strobe (CC Sink sheet)
- AC-coupled pulse limiter: TRIG (DIAG/MOSI via D3/D4) -> C16 220nF ->
  GATE-DRV, R28 10K to GND (tau 2.2 ms). 8.7-130 us strobes and the
  calibration pulse pass (guaranteed >= ~0.38 ms by the MCP1407 input
  limits); a stuck-high DIAG turns the driver off after ~1.7 ms typical,
  <= ~2.8 ms worst case, so 10 A can no longer be held on.

USB-C (Connectors sheet, USB4085-GF-A footprint)
- J2/J5 feed 5 V to the Pis: add 10K Rp on CC1/CC2 (R24-R27, 1206).
- Footprint rebuilt to GCT's land pattern (16 plated 0.40/0.66 mm pins).
  The old VBUS/GND pads had 0.1 mm top-side copper (annular-ring DRC
  errors; Pi supply current only reached them via the barrel/bottom pad).

Boost (Power sheet)
- F1 MF-MSMF050-2 polyfuse in the boost input only (+5V_BST: C1/C2/C3/R1/
  U1); PCB: +5V_BST F.Cu island, +5V B.Cu bridge keeps the Pi feed width.
- D16 P4SMA39CA clamp on VIR (open-feedback fault; relies on F1).
- R5 2K49 -> 10K (was ~0.45 W in a 1/4 W resistor).

Housekeeping
- Project sym/fp-lib-tables; USB4085-GF-A added to the symbol library;
  pin types for custom parts; locally modified Q_NPN/Q_NMOS/LED moved into
  the project library (Q_NPN_EBC, Q_NMOS_SGD, LED_ThermalPad) to keep their
  numeric pinouts; no-connect flags; PWR_FLAGs; GATE-DRV wire to Q3 fixed.
- ERC pin map (project-wide): open emitter on a power rail allowed
  (MC33063 SwE to GND).
- Add V3 Connector Only.kicad_pro (board had no rules; DRC used defaults).
- Breakaway holes marked board-only.
- Regenerated Gerber/drill zips, BOM and centroid CSVs (same for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
Parts:
- Q4: symbol Device:Q_NPN -> Pi Connector Parts:Q_NPN_EBC
Changed lines of the file:
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@@
 	)
 	(symbol
-		(lib_id "Device:Q_NPN")
+		(lib_id "Pi Connector Parts:Q_NPN_EBC")
 		(at 198.12 114.3 0)
 		(unit 1)
