File: Hardware/KiCad Source Files/V3 Connector Only.kicad_pcb (KiCad board)
At the start: 2 copper layers, 60 x 100 mm, 65 parts, among them J1 YK3210203000G, J2 USB4085-GF-A, J3 Conn_01x08, J4 YK3210203000G, J5 USB4085-GF-A, J6 USB1125-GF-B, Q1 IRLU024NPBF, Q2 IRLU024NPBF, Q3 Q_NMOS, U1 MC33063AP, U4 LM4040LP-2.0, U5 MCP4801, U6 MCP3202

Commit message: V3 connector board: strobe pulse limiter, USB-C fixes, boost protection
Mechanical: board outline, all mounting/tab/breakaway holes and every
existing part position are unchanged (checked against the previous revision);
all new parts are on the top side and no taller than existing parts.
PiTrac software compatibility: the LED current-control circuit and the
DAC/ADC/DIAG interface used by strobe_calibration_manager.py are unchanged.

Strobe (CC Sink sheet)
- AC-coupled pulse limiter: TRIG (DIAG/MOSI via D3/D4) -> C16 220nF ->
  GATE-DRV, R28 10K to GND (tau 2.2 ms). 8.7-130 us strobes and the
  calibration pulse pass (guaranteed >= ~0.38 ms by the MCP1407 input
  limits); a stuck-high DIAG turns the driver off after ~1.7 ms typical,
  <= ~2.8 ms worst case, so 10 A can no longer be held on.

USB-C (Connectors sheet, USB4085-GF-A footprint)
- J2/J5 feed 5 V to the Pis: add 10K Rp on CC1/CC2 (R24-R27, 1206).
- Footprint rebuilt to GCT's land pattern (16 plated 0.40/0.66 mm pins).
  The old VBUS/GND pads had 0.1 mm top-side copper (annular-ring DRC
  errors; Pi supply current only reached them via the barrel/bottom pad).

Boost (Power sheet)
- F1 MF-MSMF050-2 polyfuse in the boost input only (+5V_BST: C1/C2/C3/R1/
  U1); PCB: +5V_BST F.Cu island, +5V B.Cu bridge keeps the Pi feed width.
- D16 P4SMA39CA clamp on VIR (open-feedback fault; relies on F1).
- R5 2K49 -> 10K (was ~0.45 W in a 1/4 W resistor).

Housekeeping
- Project sym/fp-lib-tables; USB4085-GF-A added to the symbol library;
  pin types for custom parts; locally modified Q_NPN/Q_NMOS/LED moved into
  the project library (Q_NPN_EBC, Q_NMOS_SGD, LED_ThermalPad) to keep their
  numeric pinouts; no-connect flags; PWR_FLAGs; GATE-DRV wire to Q3 fixed.
- ERC pin map (project-wide): open emitter on a power rail allowed
  (MC33063 SwE to GND).
- Add V3 Connector Only.kicad_pro (board had no rules; DRC used defaults).
- Breakaway holes marked board-only.
- Regenerated Gerber/drill zips, BOM and centroid CSVs (same for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
Parts:
- added C16: 220nF, Capacitor_THT:C_Disc_D4.3mm_W1.9mm_P5.00mm, F.Cu at (114.0, 132.5)
- added D16: P4SMA39CA, Diode_SMD:D_SMA, F.Cu at (101.8, 93.0)
- added F1: 0.5A hold, Fuse:Fuse_1812_4532Metric_Pad1.30x3.40mm_HandSolder, F.Cu at (62.5, 105.2)
- added R24: 10K, Resistor_SMD:R_1206_3216Metric_Pad1.30x1.75mm_HandSolder, F.Cu at (69.0, 126.6)
- added R25: 10K, Resistor_SMD:R_1206_3216Metric_Pad1.30x1.75mm_HandSolder, F.Cu at (63.5, 126.6)
- added R26: 10K, Resistor_SMD:R_1206_3216Metric_Pad1.30x1.75mm_HandSolder, F.Cu at (68.0, 143.3)
- added R27: 10K, Resistor_SMD:R_1206_3216Metric_Pad1.30x1.75mm_HandSolder, F.Cu at (63.0, 143.3)
- added R28: 10K, Resistor_THT:R_Axial_DIN0207_L6.3mm_D2.5mm_P2.54mm_Vertical, F.Cu at (117.5, 130.0)
- R5: value 2K49 -> 10K
Connections:
- C1 pad 1: +5V -> +5V_BST
- C2 pad 1: +5V -> +5V_BST
- C3 pad 1: +5V -> +5V_BST
- D3 pad 1: /CC Sink/GATE-DRV -> /CC Sink/TRIG
- D4 pad 1: /CC Sink/GATE-DRV -> /CC Sink/TRIG
- R1 pad 2: +5V -> +5V_BST
- R8 pad 2: /CC Sink/GATE-DRV -> /CC Sink/TRIG
- U1 pad 6: +5V -> +5V_BST
Routing:
- net +5V_BST: track 0.00 -> 22.8 mm
- net +5V: track 18.9 -> 0.00 mm, vias 0 -> 9
- net /CC Sink/TRIG: track 0.00 -> 16.3 mm
- net /Connectors/J5_CC1: track 0.00 -> 11.0 mm
- net /Connectors/J2_CC1: track 0.00 -> 10.9 mm
- net /Connectors/J5_CC2: track 0.00 -> 8.77 mm
- net /Connectors/J2_CC2: track 0.00 -> 8.68 mm
- net VIR: track 70.5 -> 72.6 mm
- net /CC Sink/GATE-DRV: track 25.5 -> 27.2 mm, vias 0 -> 1
- net GND: vias 500 -> 486
- added copper zone on B.Cu, net +5V
- added copper zone on F.Cu, net +5V_BST

Commit message: C16: use an orderable part (K224K20X7RF5UH5, 220nF 50V X7R)
K224K15X7RF5UH5 isn't listed by any distributor; the "20" (50 V) code is the
real 220 nF part in this Vishay K series (DigiKey 2356767, element14
2860121). Footprint moved to C_Disc_D5.1mm_W3.2mm_P5.00mm, the one already
used for C2 (1 uF in the same series), so the body fits.
Outputs regenerated; ERC/DRC unchanged (0 errors), geometry unchanged.

Co-Authored-By: Claude Opus 5.5 <noreply@anthropic.com>
Parts:
- C16: footprint Capacitor_THT:C_Disc_D4.3mm_W1.9mm_P5.00mm -> Capacitor_THT:C_Disc_D5.1mm_W3.2mm_P5.00mm
